Commit message: Initial commit

File: src/robot/urdf/car.urdf.xacro (robot description, xacro)
@@ -6,16 +6,15 @@
     <gazebo>
         <plugin
-            filename="libignition-gazebo-diff-drive-system.so"
-            name="ignition::gazebo::systems::DiffDrive">
+            filename="gz-sim-diff-drive-system"
+            name="gz::sim::systems::DiffDrive">
             <left_joint>left_front_wheel_joint</left_joint>
             <left_joint>left_rear_wheel_joint</left_joint>
             <right_joint>right_front_wheel_joint</right_joint>
             <right_joint>right_rear_wheel_joint</right_joint>
-            <wheel_separation>0.4</wheel_separation>
-            <wheel_radius>0.0415</wheel_radius>
+            <wheel_separation>0.30</wheel_separation>
+            <wheel_radius>0.065</wheel_radius>
             <odom_publish_frequency>50</odom_publish_frequency>
             <frame_id>odom</frame_id>
             <child_frame_id>base_footprint</child_frame_id>
-            <topic>/cmd_vel</topic>
             <publish_wheel_tf>true</publish_wheel_tf>
             <max_linear_acceleration>10</max_linear_acceleration>
@@ -31,6 +30,6 @@
     <!-- 关节状态发布 -->
     <gazebo>
-        <plugin filename="ignition-gazebo-joint-state-publisher-system"
-        name="ignition::gazebo::systems::JointStatePublisher">
+        <plugin filename="gz-sim-joint-state-publisher-system"
+        name="gz::sim::systems::JointStatePublisher">
         </plugin>
     </gazebo>

File: src/robot/urdf/car_base.urdf.xacro (robot description, xacro)
@@ -5,12 +5,12 @@
     <!-- 定义车辆参数 -->
     <!-- 车体长宽高 -->
-    <xacro:property name="base_link_x" value="0.2"/>
-    <xacro:property name="base_link_y" value="0.12"/>
-    <xacro:property name="base_link_z" value="0.07"/>
+    <xacro:property name="base_link_x" value="0.45"/>
+    <xacro:property name="base_link_y" value="0.30"/>
+    <xacro:property name="base_link_z" value="0.16"/>
     <!-- 离地间距 -->
-    <xacro:property name="distance" value="0.015"/>
+    <xacro:property name="distance" value="0.04"/>
     <!-- 车轮半径 宽度 -->
-    <xacro:property name="wheel_radius" value="0.025"/>
-    <xacro:property name="wheel_length" value="0.02"/>
+    <xacro:property name="wheel_radius" value="0.065"/>
+    <xacro:property name="wheel_length" value="0.035"/>
     <!-- 定义颜色 -->
     <material name="yellow">

File: src/robot/urdf/car_camera.urdf.xacro (robot description, xacro)
@@ -2,7 +2,7 @@
 <robot xmlns:xacro="http://wiki.ros.org/xacro">
     <!-- 摄像头属性 -->
-    <xacro:property name="camera_x" value="0.012" /> <!-- 摄像头长度(x) -->
-    <xacro:property name="camera_y" value="0.05" /> <!-- 摄像头宽度(y) -->
-    <xacro:property name="camera_z" value="0.01" /> <!-- 摄像头高度(z) -->
+    <xacro:property name="camera_x" value="0.025" /> <!-- 摄像头长度(x) -->
+    <xacro:property name="camera_y" value="0.06" /> <!-- 摄像头宽度(y) -->
+    <xacro:property name="camera_z" value="0.025" /> <!-- 摄像头高度(z) -->
     <xacro:property name="camera_joint_x" value="${base_link_x / 2 - camera_x / 2}" /> <!-- 摄像头安装的x坐标 -->
     <xacro:property name="camera_joint_y" value="0.0" /> <!-- 摄像头安装的y坐标 -->

File: src/robot/urdf/car_laser.urdf.xacro (robot description, xacro)
@@ -7,6 +7,6 @@
     </material>
     <!-- 雷达属性 -->
-    <xacro:property name="laser_length" value="0.03" /> <!-- 雷达长度 -->
-    <xacro:property name="laser_radius" value="0.03" /> <!-- 雷达半径 -->
+    <xacro:property name="laser_length" value="0.05" /> <!-- 雷达长度 -->
+    <xacro:property name="laser_radius" value="0.05" /> <!-- 雷达半径 -->
     <xacro:property name="laser_joint_x" value="0.0" /> <!-- 雷达安装的x坐标 -->
     <xacro:property name="laser_joint_y" value="0.0" /> <!-- 雷达安装的y坐标 -->
@@ -27,3 +27,31 @@
         <origin xyz="${laser_joint_x} ${laser_joint_y} ${laser_joint_z}" />
     </joint>
+    <gazebo reference="laser">
+        <sensor name="laser_sensor" type="gpu_lidar">
+            <topic>/scan</topic>
+            <update_rate>10</update_rate>
+            <ray>
+                <scan>
+                    <horizontal>
+                        <samples>360</samples>
+                        <resolution>1</resolution>
+                        <min_angle>-${PI}</min_angle>
+                        <max_angle>${PI}</max_angle>
+                    </horizontal>
+                </scan>
+                <range>
+                    <min>0.12</min>
+                    <max>8.0</max>
+                    <resolution>0.01</resolution>
+                </range>
+                <noise>
+                    <type>gaussian</type>
+                    <mean>0.0</mean>
+                    <stddev>0.01</stddev>
+                </noise>
+            </ray>
+            <always_on>true</always_on>
+            <visualize>true</visualize>
+        </sensor>
+    </gazebo>
 </robot>

Commit message: Tune simulation SLAM and robot model

File: src/robot/urdf/car.urdf.xacro (robot description, xacro)
@@ -9,7 +9,5 @@
             name="gz::sim::systems::DiffDrive">
             <left_joint>left_front_wheel_joint</left_joint>
-            <left_joint>left_rear_wheel_joint</left_joint>
             <right_joint>right_front_wheel_joint</right_joint>
-            <right_joint>right_rear_wheel_joint</right_joint>
             <wheel_separation>0.30</wheel_separation>
             <wheel_radius>0.065</wheel_radius>
@@ -18,12 +16,12 @@
             <child_frame_id>base_footprint</child_frame_id>
             <publish_wheel_tf>true</publish_wheel_tf>
-            <max_linear_acceleration>10</max_linear_acceleration>
-            <min_linear_acceleration>-10</min_linear_acceleration>
-            <max_angular_acceleration>10</max_angular_acceleration>
-            <min_angular_acceleration>-10</min_angular_acceleration>
-            <max_linear_velocity>0.5</max_linear_velocity>
-            <min_linear_velocity>-0.5</min_linear_velocity>
-            <max_angular_velocity>1</max_angular_velocity>
-            <min_angular_velocity>-1</min_angular_velocity>
+            <max_linear_acceleration>0.35</max_linear_acceleration>
+            <min_linear_acceleration>-0.35</min_linear_acceleration>
+            <max_angular_acceleration>0.8</max_angular_acceleration>
+            <min_angular_acceleration>-0.8</min_angular_acceleration>
+            <max_linear_velocity>0.35</max_linear_velocity>
+            <min_linear_velocity>-0.35</min_linear_velocity>
+            <max_angular_velocity>0.8</max_angular_velocity>
+            <min_angular_velocity>-0.8</min_angular_velocity>
         </plugin>
     </gazebo>

File: src/robot/urdf/car_base.urdf.xacro (robot description, xacro)
@@ -49,5 +49,5 @@
             <material name="yellow"/>
         </collision>
-        <xacro:box_inertia m="1.0" w="${base_link_x}" d="${base_link_y}" h="${base_link_z}"/>
+        <xacro:box_inertia m="5.0" w="${base_link_x}" d="${base_link_y}" h="${base_link_z}"/>
     </link>
     <joint name="baselink2basefootprint" type="fixed">
@@ -73,5 +73,5 @@
                 <material name="gray"/>
             </collision>
-            <xacro:cylinder_inertia m="1.0" r="${wheel_radius}" h="${wheel_length}"/>
+            <xacro:cylinder_inertia m="0.15" r="${wheel_radius}" h="${wheel_length}"/>
         </link>
         <joint name="${wheel_name}_wheel_joint" type="continuous">
@@ -80,10 +80,48 @@
             <origin xyz="${(base_link_x / 2 - wheel_radius) * is_front} ${base_link_y / 2 * is_left} ${(base_link_z / 2 + distance - wheel_radius) * -1}" rpy="0 0 0" />
             <axis xyz="0 1 0" />
+            <dynamics damping="0.08" friction="0.01" />
         </joint>
     </xacro:macro>
-    <!-- 车轮宏调用 -->
-    <xacro:wheel_func wheel_name="left_front" is_front="1" is_left="1" />
-    <xacro:wheel_func wheel_name="left_rear" is_front="-1" is_left="1" />
-    <xacro:wheel_func wheel_name="right_front" is_front="1" is_left="-1" />
-    <xacro:wheel_func wheel_name="right_rear" is_front="-1" is_left="-1" />
+    <xacro:macro name="wheel_friction" params="wheel_name">
+        <gazebo reference="${wheel_name}_wheel">
+            <mu1>1.0</mu1>
+            <mu2>0.25</mu2>
+            <kp>1000000.0</kp>
+            <kd>10.0</kd>
+        </gazebo>
+    </xacro:macro>
+    <xacro:macro name="caster_func" params="caster_name is_front">
+        <link name="${caster_name}_caster">
+            <visual>
+                <geometry>
+                    <sphere radius="0.035" />
+                </geometry>
+                <material name="gray" />
+            </visual>
+            <collision>
+                <geometry>
+                    <sphere radius="0.035" />
+                </geometry>
+            </collision>
+            <xacro:sphere_inertia m="0.05" r="0.035" />
+        </link>
+        <joint name="${caster_name}_caster_joint" type="fixed">
+            <parent link="base_link" />
+            <child link="${caster_name}_caster" />
+            <origin xyz="${(base_link_x / 2 - 0.08) * is_front} 0 ${(base_link_z / 2 + distance - 0.035) * -1}" rpy="0 0 0" />
+        </joint>
+        <gazebo reference="${caster_name}_caster">
+            <mu1>0.05</mu1>
+            <mu2>0.05</mu2>
+            <kp>1000000.0</kp>
+            <kd>10.0</kd>
+        </gazebo>
+    </xacro:macro>
+    <!-- Two centered drive wheels plus low-friction front/rear supports. -->
+    <xacro:wheel_func wheel_name="left_front" is_front="0" is_left="1" />
+    <xacro:wheel_func wheel_name="right_front" is_front="0" is_left="-1" />
+    <xacro:wheel_friction wheel_name="left_front" />
+    <xacro:wheel_friction wheel_name="right_front" />
+    <xacro:caster_func caster_name="front" is_front="1" />
+    <xacro:caster_func caster_name="rear" is_front="-1" />
 </robot>
